File: TENG_loads-main/TENG_loads-main/Project/load_automatisation.kicad_pcb (KiCad board)
At the start: 2 copper layers, 263.4 x 251.4 mm, 123 parts, among them IC1 OPA2145IDR, IC10 TBD62083AFG, IC11 74HC238D,653, IC2 TBD62083AFG, IC3 TBD62083AFG, IC4 74HC238D,653, IC5 74HC238D,653, IC6 TBD62083AFG, IC7 TBD62083AFG, IC8 TBD62083AFG, IC9 OPA145IDBVT, J1 PowerNeg, J12 PH-2X05SG, J13 1757242, J30 1757349, J9 PowerIn, K1 V23079C1103B301, K10 IMC03TS, K11 V23079C1103B301, K12 V23079C1103B301, K13 V23079C1103B301, K14 IMC03TS, K15 IMC03TS, K16 IMC03TS, K17 V23079C1103B301, K18 V23079C1103B301, K19 V23079C1103B301, K2 V23079C1103B301, K20 V23079C1103B301, K21 V23079C1103B301, K22 IMC03TS, K23 IMC03TS, K24 IMC03TS, K25 IMC03TS, K26 IMC03TS, K27 V23079C1103B301, K28 V23079C1103B301, K29 V23079C1103B301, K3 V23079C1103B301, K30 IMC03TS, K31 IMC03TS, K32 IMC03TS, K33 V23079C1103B301, K34 V23079C1103B301, K35 V23079C1103B301, K36 V23079C1103B301, K37 V23079C1103B301, K38 IMC03TS, K39 IMC03TS, K4 V23079C1103B301, K40 IMC03TS, K41 IMC03TS, K42 IMC03TS, K43 V23079C1103B301, K44 V23079C1103B301, K45 V23079C1103B301, K46 IMC03TS, K47 IMC03TS, K48 IMC03TS, K5 V23079C1103B301, K6 IMC03TS, K7 IMC03TS, K8 IMC03TS, K9 IMC03TS, U1 AMS1117-5.0, U2 INA128, U3 AMS1117-5.0

Commit message: Updated connections
Parts:
- removed J9: PowerIn, Connector_PinHeader_2.54mm:PinHeader_1x02_P2.54mm_Vertical
- added J2: 1757242, SamacSys_Parts:1757242, F.Cu at (91.4, 168.5)
- added J3: 1757242, SamacSys_Parts:1757242, F.Cu at (91.3, 150.2)
- added J4: PowerIn, Connector_PinHeader_2.54mm:PinHeader_1x02_P2.54mm_Vertical, F.Cu at (111.6, 173.8)
- C1, C15: value 100uF -> 10uF
- C16, C2: value 100uF -> 22uF
- K1, K11, K12, K13, K17, K18, K19, K2, K20, K21, K27, K28, K29, K3, K33, K34, K35, K36, K37, K4, K43, K44, K45, K5: value V23079C1103B301 -> V23079A1001B301
- moved J1 14.3 mm to (109.5, 157.6), turned to -90 degrees
Connections:
- J1 pad 2: GND -> Net-(J1-Pin_2)
- J12 pad 1: /Teng- -> /TengN_sw
- J12 pad 2: /TengN -> /TengN_IN
- J12 pad 3: /Teng- -> /TengN_sw
- J12 pad 5: /Teng- -> /TengN_sw
- J12 pad 7: /TengN -> /TengN_IN
- J13 pad 2: /TengN -> /Teng-
- K1 pad 5: /Teng+ -> /TengP_IN
- K10 pad 5: /Teng- -> /TengN_sw
- K11 pad 5: /Teng+ -> /TengP_IN
- K12 pad 5: /Teng+ -> /TengP_IN
- K13 pad 5: /Teng+ -> /TengP_IN
- K14 pad 5: /Teng- -> /TengN_sw
- K15 pad 5: /Teng- -> /TengN_sw
- K16 pad 5: /Teng- -> /TengN_sw
- K17 pad 5: /Teng+ -> /TengP_IN
- K18 pad 5: /Teng+ -> /TengP_IN
- K19 pad 5: /Teng+ -> /TengP_IN
- K2 pad 5: /Teng+ -> /TengP_IN
- K20 pad 5: /Teng+ -> /TengP_IN
- K21 pad 5: /Teng+ -> /TengP_IN
- K22 pad 5: /Teng- -> /TengN_sw
- K23 pad 5: /Teng- -> /TengN_sw
- K24 pad 5: /Teng- -> /TengN_sw
- K25 pad 5: /Teng- -> /TengN_sw
- K26 pad 5: /Teng- -> /TengN_sw
- K27 pad 5: /Teng+ -> /TengP_IN
- K28 pad 5: /Teng+ -> /TengP_IN
- K29 pad 5: /Teng+ -> /TengP_IN
- K3 pad 5: /Teng+ -> /TengP_IN
- K30 pad 5: /Teng- -> /TengN_sw
- K31 pad 5: /Teng- -> /TengN_sw
- K32 pad 5: /Teng- -> /TengN_sw
- K33 pad 5: /Teng+ -> /TengP_IN
- K34 pad 5: /Teng+ -> /TengP_IN
- K35 pad 5: /Teng+ -> /TengP_IN
- K36 pad 5: /Teng+ -> /TengP_IN
- K37 pad 5: /Teng+ -> /TengP_IN
- K38 pad 5: /Teng- -> /TengN_sw
- K39 pad 5: /Teng- -> /TengN_sw
- K4 pad 5: /Teng+ -> /TengP_IN
- K40 pad 5: /Teng- -> /TengN_sw
- K41 pad 5: /Teng- -> /TengN_sw
- K42 pad 5: /Teng- -> /TengN_sw
- K43 pad 5: /Teng+ -> /TengP_IN
- K44 pad 5: /Teng+ -> /TengP_IN
- K45 pad 5: /Teng+ -> /TengP_IN
- K46 pad 5: /Teng- -> /TengN_sw
- K47 pad 5: /Teng- -> /TengN_sw
- K48 pad 5: /Teng- -> /TengN_sw
- K5 pad 5: /Teng+ -> /TengP_IN
- K6 pad 5: /Teng- -> /TengN_sw
- K7 pad 5: /Teng- -> /TengN_sw
- K8 pad 5: /Teng- -> /TengN_sw
- K9 pad 5: /Teng- -> /TengN_sw
- TENG_Connector1 pad 1: /Teng+ -> /TengP_IN
- TENG_Connector1 pad 3: /TengN -> /Teng-
- TENG_Connector1 pad 4: /TengN -> /TengN_IN
- TENG_Connector2 pad 1: unconnected-(TENG_Connector2-Pin_1-Pad1) -> /TengP_IN
- TENG_Connector2 pad 2: unconnected-(TENG_Connector2-Pin_2-Pad2) -> /Teng+
- TENG_Connector2 pad 3: unconnected-(TENG_Connector2-Pin_3-Pad3) -> /Teng-
- TENG_Connector2 pad 4: unconnected-(TENG_Connector2-Pin_4-Pad4) -> /TengN_IN
Routing:
- net /TengP_IN: track 0.00 -> 896.7 mm, vias 0 -> 22
- net /Teng+: track 926.1 -> 36.0 mm, vias 22 -> 0
- net /TengN: track 78.3 -> 0.00 mm
- net /TengN_IN: track 0.00 -> 47.1 mm
- net /Teng-: track 875.1 -> 839.0 mm
- net /TengN_sw: track 0.00 -> 35.6 mm
- net GND: track 808.4 -> 793.2 mm
