File: TENG_Loads_PCB/1_Loads.kicad_sch (KiCad schematic)
At the start: 9 parts, among them IC11 74HC238D,653, IC2 TBD62083AFG, IC3 TBD62083AFG

Commit message: Update footprints
Update component footprints, and advancing in the design.
Parts:
- IC2, IC3: footprint SamacSys_Parts:SOIC127P1030X245-18N -> TENG_Footprint_Library:SOIC127P1030X245-18N
Changed lines of the file:
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@@
 			)
 		)
-		(property "Footprint" "SamacSys_Parts:SOIC127P1030X245-18N"
+		(property "Footprint" "TENG_Footprint_Library:SOIC127P1030X245-18N"
 			(at 167.64 129.21 0)
 			(hide yes)
@@
 			)
 		)
-		(property "Footprint" "SamacSys_Parts:SOIC127P1030X245-18N"
+		(property "Footprint" "TENG_Footprint_Library:SOIC127P1030X245-18N"
 			(at 120.65 129.21 0)
 			(hide yes)
