File: TENG_Loads_PCB/2_Loads.kicad_sch (KiCad schematic)
At the start: 9 parts, among them IC4 74HC238D,653, IC6 TBD62083AFG, IC7 TBD62083AFG

Commit message: Update footprints
Update component footprints, and advancing in the design.
Parts:
- IC6, IC7: footprint SamacSys_Parts:SOIC127P1030X245-18N -> TENG_Footprint_Library:SOIC127P1030X245-18N
Changed lines of the file:
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@@
 			)
 		)
-		(property "Footprint" "SamacSys_Parts:SOIC127P1030X245-18N"
+		(property "Footprint" "TENG_Footprint_Library:SOIC127P1030X245-18N"
 			(at 190.5 124.13 0)
 			(hide yes)
@@
 			)
 		)
-		(property "Footprint" "SamacSys_Parts:SOIC127P1030X245-18N"
+		(property "Footprint" "TENG_Footprint_Library:SOIC127P1030X245-18N"
 			(at 138.43 124.13 0)
 			(hide yes)
