File: TENG_Loads_PCB/Loads-1.kicad_sch (KiCad schematic)
At the start: 24 parts, among them K1 V23079A1001B301, K10 IMC03TS, K11 V23079A1001B301, K12 V23079A1001B301, K13 V23079A1001B301, K14 IMC03TS, K15 IMC03TS, K16 IMC03TS, K2 V23079A1001B301, K3 V23079A1001B301, K4 V23079A1001B301, K5 V23079A1001B301, K6 IMC03TS, K7 IMC03TS, K8 IMC03TS, K9 IMC03TS

Commit message: Update footprints
Update component footprints, and advancing in the design.
Parts:
- K1, K11, K12, K13, K2, K3, K4, K5: footprint SamacSys_Parts:V23079A1001B301 -> TENG_Footprint_Library:V23079A1001B301
- K10, K14, K15, K16, K6, K7, K8, K9: footprint SamacSys_Parts:IMC03TS -> TENG_Footprint_Library:IMC03TS
Changed lines of the file:
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@@
 			)
 		)
-		(property "Footprint" "SamacSys_Parts:V23079A1001B301"
+		(property "Footprint" "TENG_Footprint_Library:V23079A1001B301"
 			(at 115.57 171.12 0)
 			(hide yes)
@@
 			)
 		)
-		(property "Footprint" "SamacSys_Parts:V23079A1001B301"
+		(property "Footprint" "TENG_Footprint_Library:V23079A1001B301"
 			(at 118.11 280.34 0)
 			(hide yes)
@@
 			)
 		)
-		(property "Footprint" "SamacSys_Parts:V23079A1001B301"
+		(property "Footprint" "TENG_Footprint_Library:V23079A1001B301"
 			(at 255.27 214.3 0)
 			(hide yes)
@@
 			)
 		)
-		(property "Footprint" "SamacSys_Parts:IMC03TS"
+		(property "Footprint" "TENG_Footprint_Library:IMC03TS"
 			(at 96.52 115.24 0)
 			(hide yes)
@@
 			)
 		)
-		(property "Footprint" "SamacSys_Parts:V23079A1001B301"
+		(property "Footprint" "TENG_Footprint_Library:V23079A1001B301"
 			(at 115.57 243.51 0)
 			(hide yes)
@@
 			)
 		)
-		(property "Footprint" "SamacSys_Parts:IMC03TS"
+		(property "Footprint" "TENG_Footprint_Library:IMC03TS"
 			(at 96.52 154.61 0)
 			(hide yes)
@@
 			)
 		)
-		(property "Footprint" "SamacSys_Parts:V23079A1001B301"
+		(property "Footprint" "TENG_Footprint_Library:V23079A1001B301"
 			(at 257.81 134.29 0)
 			(hide yes)
@@
 			)
 		)
-		(property "Footprint" "SamacSys_Parts:IMC03TS"
+		(property "Footprint" "TENG_Footprint_Library:IMC03TS"
 			(at 96.52 191.44 0)
 			(hide yes)
@@
 			)
 		)
-		(property "Footprint" "SamacSys_Parts:V23079A1001B301"
+		(property "Footprint" "TENG_Footprint_Library:V23079A1001B301"
 			(at 255.27 174.93 0)
 			(hide yes)
@@
 			)
 		)
-		(property "Footprint" "SamacSys_Parts:V23079A1001B301"
+		(property "Footprint" "TENG_Footprint_Library:V23079A1001B301"
 			(at 115.57 207.95 0)
 			(hide yes)
@@
 			)
 		)
-		(property "Footprint" "SamacSys_Parts:IMC03TS"
+		(property "Footprint" "TENG_Footprint_Library:IMC03TS"
 			(at 96.52 227 0)
 			(hide yes)
@@
 			)
 		)
-		(property "Footprint" "SamacSys_Parts:IMC03TS"
+		(property "Footprint" "TENG_Footprint_Library:IMC03TS"
 			(at 238.76 117.78 0)
 			(hide yes)
@@
 			)
 		)
-		(property "Footprint" "SamacSys_Parts:IMC03TS"
+		(property "Footprint" "TENG_Footprint_Library:IMC03TS"
 			(at 99.06 263.83 0)
 			(hide yes)
@@
 			)
 		)
-		(property "Footprint" "SamacSys_Parts:IMC03TS"
+		(property "Footprint" "TENG_Footprint_Library:IMC03TS"
 			(at 236.22 158.42 0)
 			(hide yes)
@@
 			)
 		)
-		(property "Footprint" "SamacSys_Parts:IMC03TS"
+		(property "Footprint" "TENG_Footprint_Library:IMC03TS"
 			(at 236.22 197.79 0)
 			(hide yes)
@@
 			)
 		)
-		(property "Footprint" "SamacSys_Parts:V23079A1001B301"
+		(property "Footprint" "TENG_Footprint_Library:V23079A1001B301"
 			(at 115.57 131.75 0)
 			(hide yes)
