File: TENG_Loads_PCB/Loads-2.kicad_sch (KiCad schematic)
At the start: 24 parts, among them K17 V23079A1001B301, K18 V23079A1001B301, K19 V23079A1001B301, K20 V23079A1001B301, K21 V23079A1001B301, K22 IMC03TS, K23 IMC03TS, K24 IMC03TS, K25 IMC03TS, K26 IMC03TS, K27 V23079A1001B301, K28 V23079A1001B301, K29 V23079A1001B301, K30 IMC03TS, K31 IMC03TS, K32 IMC03TS

Commit message: Update footprints
Update component footprints, and advancing in the design.
Parts:
- K17, K18, K19, K20, K21, K27, K28, K29: footprint SamacSys_Parts:V23079A1001B301 -> TENG_Footprint_Library:V23079A1001B301
- K22, K23, K24, K25, K26, K30, K31, K32: footprint SamacSys_Parts:IMC03TS -> TENG_Footprint_Library:IMC03TS
Changed lines of the file:
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@@
 			)
 		)
-		(property "Footprint" "SamacSys_Parts:V23079A1001B301"
+		(property "Footprint" "TENG_Footprint_Library:V23079A1001B301"
 			(at 115.57 171.12 0)
 			(hide yes)
@@
 			)
 		)
-		(property "Footprint" "SamacSys_Parts:V23079A1001B301"
+		(property "Footprint" "TENG_Footprint_Library:V23079A1001B301"
 			(at 118.11 280.34 0)
 			(hide yes)
@@
 			)
 		)
-		(property "Footprint" "SamacSys_Parts:V23079A1001B301"
+		(property "Footprint" "TENG_Footprint_Library:V23079A1001B301"
 			(at 255.27 214.3 0)
 			(hide yes)
@@
 			)
 		)
-		(property "Footprint" "SamacSys_Parts:IMC03TS"
+		(property "Footprint" "TENG_Footprint_Library:IMC03TS"
 			(at 96.52 115.24 0)
 			(hide yes)
@@
 			)
 		)
-		(property "Footprint" "SamacSys_Parts:V23079A1001B301"
+		(property "Footprint" "TENG_Footprint_Library:V23079A1001B301"
 			(at 115.57 243.51 0)
 			(hide yes)
@@
 			)
 		)
-		(property "Footprint" "SamacSys_Parts:IMC03TS"
+		(property "Footprint" "TENG_Footprint_Library:IMC03TS"
 			(at 96.52 154.61 0)
 			(hide yes)
@@
 			)
 		)
-		(property "Footprint" "SamacSys_Parts:V23079A1001B301"
+		(property "Footprint" "TENG_Footprint_Library:V23079A1001B301"
 			(at 257.81 134.29 0)
 			(hide yes)
@@
 			)
 		)
-		(property "Footprint" "SamacSys_Parts:IMC03TS"
+		(property "Footprint" "TENG_Footprint_Library:IMC03TS"
 			(at 96.52 191.44 0)
 			(hide yes)
@@
 			)
 		)
-		(property "Footprint" "SamacSys_Parts:V23079A1001B301"
+		(property "Footprint" "TENG_Footprint_Library:V23079A1001B301"
 			(at 255.27 174.93 0)
 			(hide yes)
@@
 			)
 		)
-		(property "Footprint" "SamacSys_Parts:V23079A1001B301"
+		(property "Footprint" "TENG_Footprint_Library:V23079A1001B301"
 			(at 115.57 207.95 0)
 			(hide yes)
@@
 			)
 		)
-		(property "Footprint" "SamacSys_Parts:IMC03TS"
+		(property "Footprint" "TENG_Footprint_Library:IMC03TS"
 			(at 96.52 227 0)
 			(hide yes)
@@
 			)
 		)
-		(property "Footprint" "SamacSys_Parts:IMC03TS"
+		(property "Footprint" "TENG_Footprint_Library:IMC03TS"
 			(at 238.76 117.78 0)
 			(hide yes)
@@
 			)
 		)
-		(property "Footprint" "SamacSys_Parts:IMC03TS"
+		(property "Footprint" "TENG_Footprint_Library:IMC03TS"
 			(at 99.06 263.83 0)
 			(hide yes)
@@
 			)
 		)
-		(property "Footprint" "SamacSys_Parts:IMC03TS"
+		(property "Footprint" "TENG_Footprint_Library:IMC03TS"
 			(at 236.22 158.42 0)
 			(hide yes)
@@
 			)
 		)
-		(property "Footprint" "SamacSys_Parts:IMC03TS"
+		(property "Footprint" "TENG_Footprint_Library:IMC03TS"
 			(at 236.22 197.79 0)
 			(hide yes)
@@
 			)
 		)
-		(property "Footprint" "SamacSys_Parts:V23079A1001B301"
+		(property "Footprint" "TENG_Footprint_Library:V23079A1001B301"
 			(at 115.57 131.75 0)
 			(hide yes)
