File: TENG_Loads_PCB/Loads-3.kicad_sch (KiCad schematic)
At the start: 24 parts, among them K33 V23079A1001B301, K34 V23079A1001B301, K35 V23079A1001B301, K36 V23079A1001B301, K37 V23079A1001B301, K38 IMC03TS, K39 IMC03TS, K40 IMC03TS, K41 IMC03TS, K42 IMC03TS, K43 V23079A1001B301, K44 V23079A1001B301, K45 V23079A1001B301, K46 IMC03TS, K47 IMC03TS, K48 IMC03TS

Commit message: Update footprints
Update component footprints, and advancing in the design.
Parts:
- K33, K34, K35, K36, K37, K43, K44, K45: footprint SamacSys_Parts:V23079A1001B301 -> TENG_Footprint_Library:V23079A1001B301
- K38, K39, K40, K41, K42, K46, K47, K48: footprint SamacSys_Parts:IMC03TS -> TENG_Footprint_Library:IMC03TS
Changed lines of the file:
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@@
 			)
 		)
-		(property "Footprint" "SamacSys_Parts:V23079A1001B301"
+		(property "Footprint" "TENG_Footprint_Library:V23079A1001B301"
 			(at 115.57 171.12 0)
 			(hide yes)
@@
 			)
 		)
-		(property "Footprint" "SamacSys_Parts:V23079A1001B301"
+		(property "Footprint" "TENG_Footprint_Library:V23079A1001B301"
 			(at 118.11 280.34 0)
 			(hide yes)
@@
 			)
 		)
-		(property "Footprint" "SamacSys_Parts:V23079A1001B301"
+		(property "Footprint" "TENG_Footprint_Library:V23079A1001B301"
 			(at 255.27 214.3 0)
 			(hide yes)
@@
 			)
 		)
-		(property "Footprint" "SamacSys_Parts:IMC03TS"
+		(property "Footprint" "TENG_Footprint_Library:IMC03TS"
 			(at 96.52 115.24 0)
 			(hide yes)
@@
 			)
 		)
-		(property "Footprint" "SamacSys_Parts:V23079A1001B301"
+		(property "Footprint" "TENG_Footprint_Library:V23079A1001B301"
 			(at 115.57 243.51 0)
 			(hide yes)
@@
 			)
 		)
-		(property "Footprint" "SamacSys_Parts:IMC03TS"
+		(property "Footprint" "TENG_Footprint_Library:IMC03TS"
 			(at 96.52 154.61 0)
 			(hide yes)
@@
 			)
 		)
-		(property "Footprint" "SamacSys_Parts:V23079A1001B301"
+		(property "Footprint" "TENG_Footprint_Library:V23079A1001B301"
 			(at 257.81 134.29 0)
 			(hide yes)
@@
 			)
 		)
-		(property "Footprint" "SamacSys_Parts:IMC03TS"
+		(property "Footprint" "TENG_Footprint_Library:IMC03TS"
 			(at 96.52 191.44 0)
 			(hide yes)
@@
 			)
 		)
-		(property "Footprint" "SamacSys_Parts:V23079A1001B301"
+		(property "Footprint" "TENG_Footprint_Library:V23079A1001B301"
 			(at 255.27 174.93 0)
 			(hide yes)
@@
 			)
 		)
-		(property "Footprint" "SamacSys_Parts:V23079A1001B301"
+		(property "Footprint" "TENG_Footprint_Library:V23079A1001B301"
 			(at 115.57 207.95 0)
 			(hide yes)
@@
 			)
 		)
-		(property "Footprint" "SamacSys_Parts:IMC03TS"
+		(property "Footprint" "TENG_Footprint_Library:IMC03TS"
 			(at 96.52 227 0)
 			(hide yes)
@@
 			)
 		)
-		(property "Footprint" "SamacSys_Parts:IMC03TS"
+		(property "Footprint" "TENG_Footprint_Library:IMC03TS"
 			(at 238.76 117.78 0)
 			(hide yes)
@@
 			)
 		)
-		(property "Footprint" "SamacSys_Parts:IMC03TS"
+		(property "Footprint" "TENG_Footprint_Library:IMC03TS"
 			(at 99.06 263.83 0)
 			(hide yes)
@@
 			)
 		)
-		(property "Footprint" "SamacSys_Parts:IMC03TS"
+		(property "Footprint" "TENG_Footprint_Library:IMC03TS"
 			(at 236.22 158.42 0)
 			(hide yes)
@@
 			)
 		)
-		(property "Footprint" "SamacSys_Parts:IMC03TS"
+		(property "Footprint" "TENG_Footprint_Library:IMC03TS"
 			(at 236.22 197.79 0)
 			(hide yes)
@@
 			)
 		)
-		(property "Footprint" "SamacSys_Parts:V23079A1001B301"
+		(property "Footprint" "TENG_Footprint_Library:V23079A1001B301"
 			(at 115.57 131.75 0)
 			(hide yes)
