File: TENG_Loads_PCB/load_automatisation.kicad_pcb (KiCad board)
At the start: 2 copper layers, 263.4 x 251.4 mm, 131 parts, among them IC1 OPA2145IDR, IC10 TBD62083AFG, IC11 74HC238D,653, IC2 TBD62083AFG, IC3 TBD62083AFG, IC4 74HC238D,653, IC5 74HC238D,653, IC6 TBD62083AFG, IC7 TBD62083AFG, IC8 TBD62083AFG, IC9 OPA145IDBVT, J1 PowerNeg, J12 PH-2X05SG, J13 1757242, J2 1757242, J3 1757242, J30 1757349, J4 PowerIn, K1 V23079C1103B301, K10 IMC03TS, K11 V23079C1103B301, K12 V23079C1103B301, K13 V23079C1103B301, K14 IMC03TS, K15 IMC03TS, K16 IMC03TS, K17 V23079C1103B301, K18 V23079C1103B301, K19 V23079C1103B301, K2 V23079C1103B301, K20 V23079C1103B301, K21 V23079C1103B301, K22 IMC03TS, K23 IMC03TS, K24 IMC03TS, K25 IMC03TS, K26 IMC03TS, K27 V23079C1103B301, K28 V23079C1103B301, K29 V23079C1103B301, K3 V23079C1103B301, K30 IMC03TS, K31 IMC03TS, K32 IMC03TS, K33 V23079C1103B301, K34 V23079C1103B301, K35 V23079C1103B301, K36 V23079C1103B301, K37 V23079C1103B301, K38 IMC03TS, K39 IMC03TS, K4 V23079C1103B301, K40 IMC03TS, K41 IMC03TS, K42 IMC03TS, K43 V23079C1103B301, K44 V23079C1103B301, K45 V23079C1103B301, K46 IMC03TS, K47 IMC03TS, K48 IMC03TS, K5 V23079C1103B301, K6 IMC03TS, K7 IMC03TS, K8 IMC03TS, K9 IMC03TS, U1 AMS1117-5.0, U2 INA128, U3 AMS1117-5.0

Commit message: Update footprints
Update component footprints, and advancing in the design.
Parts:
- removed C15: 10uF, Capacitor_THT:CP_Radial_D8.0mm_P3.80mm
- removed C16: 22uF, Capacitor_THT:CP_Radial_D8.0mm_P3.80mm
- removed C17, C18, C19, C20, C3, C4, C5: 100nF, Capacitor_SMD:C_0805_2012Metric
- removed IC1: OPA2145IDR, Library:SOIC127P600X175-8N
- removed IC9: OPA145IDBVT, Library:SOT95P280X145-5N
- removed J12: PH-2X05SG, SamacSys_Parts:HDRV10W66P254_2X5_1270X500X895P
- removed J3: 1757242, Library:1757242
- removed J30: 1757349, Library:SHDRRA12W103P0X508_1X12_6296X1200X875P
- removed R1, R3, R4: R, Resistor_SMD:R_0805_2012Metric
- removed U2: INA128, Package_SO:SOIC-8_3.9x4.9mm_P1.27mm
- removed U3: AMS1117-5.0, Package_TO_SOT_SMD:SOT-223-3_TabPin2
- IC10, IC2, IC3, IC6, IC7, IC8: footprint Library:SOIC127P1030X245-18N -> TENG_Footprint_Library:SOIC127P1030X245-18N
- IC11, IC4, IC5: footprint Library:74HC238D653 -> TENG_Footprint_Library:74HC238D653
- J1: value PowerNeg -> 1923937; footprint Connector_PinHeader_2.54mm:PinHeader_1x02_P2.54mm_Vertical -> TENG_Footprint_Library:1923937
- J13, J2: footprint Library:1757242 -> TENG_Footprint_Library:1757242
- K1, K11, K12, K13, K17, K18, K19, K2, K20, K21, K27, K28, K29, K3, K33, K34, K35, K36, K37, K4, K43, K44, K45, K5: value V23079C1103B301 -> V23079A1001B301; footprint Library:V23079A1001B301 -> TENG_Footprint_Library:V23079A1001B301
- K10, K14, K15, K16, K22, K23, K24, K25, K26, K30, K31, K32, K38, K39, K40, K41, K42, K46, K47, K48, K6, K7, K8, K9: footprint Library:IMC03TS -> TENG_Footprint_Library:IMC03TS
- moved J1 47.7 mm to (128.5, 203.2), turned to -90 degrees
- moved C2 3.81 mm to (168.5, 169.7), turned to -90 degrees
- moved C1 3.65 mm to (146.0, 169.2), turned to -90 degrees
- moved J4 2.65 mm to (137.5, 169.0)
- moved J2 0.21 mm to (128.5, 169.0)
Connections:
- J1 pad 1: /VNeg -> GND
- J1 pad 2: Net-(J1-Pin_2) -> /Din0
- J2 pad 1: GND -> Net-(J4-Pin_1)
- J2 pad 2: Net-(J4-Pin_2) -> GND
- J4 pad 1: /Vin -> Net-(J4-Pin_1)
- J4 pad 2: Net-(J4-Pin_2) -> /Vin
- K1 pad 8: /Vsense -> /V_daq+
- K10 pad 5: /TengN_sw -> /TengN_IN
- K11 pad 8: /Vsense -> /V_daq+
- K12 pad 8: /Vsense -> /V_daq+
- K13 pad 8: /Vsense -> /V_daq+
- K14 pad 5: /TengN_sw -> /TengN_IN
- K15 pad 5: /TengN_sw -> /TengN_IN
- K16 pad 5: /TengN_sw -> /TengN_IN
- K17 pad 8: /Vsense -> /V_daq+
- K18 pad 8: /Vsense -> /V_daq+
- K19 pad 8: /Vsense -> /V_daq+
- K2 pad 8: /Vsense -> /V_daq+
- K20 pad 8: /Vsense -> /V_daq+
- K21 pad 8: /Vsense -> /V_daq+
- K22 pad 5: /TengN_sw -> /TengN_IN
- K23 pad 5: /TengN_sw -> /TengN_IN
- K24 pad 5: /TengN_sw -> /TengN_IN
- K25 pad 5: /TengN_sw -> /TengN_IN
- K26 pad 5: /TengN_sw -> /TengN_IN
- K27 pad 8: /Vsense -> /V_daq+
- K28 pad 8: /Vsense -> /V_daq+
- K29 pad 8: /Vsense -> /V_daq+
- K3 pad 8: /Vsense -> /V_daq+
- K30 pad 5: /TengN_sw -> /TengN_IN
- K31 pad 5: /TengN_sw -> /TengN_IN
- K32 pad 5: /TengN_sw -> /TengN_IN
- K33 pad 8: /Vsense -> /V_daq+
- K34 pad 8: /Vsense -> /V_daq+
- K35 pad 8: /Vsense -> /V_daq+
- K36 pad 8: /Vsense -> /V_daq+
- K37 pad 8: /Vsense -> /V_daq+
- K38 pad 5: /TengN_sw -> /TengN_IN
- K39 pad 5: /TengN_sw -> /TengN_IN
- K4 pad 8: /Vsense -> /V_daq+
- K40 pad 5: /TengN_sw -> /TengN_IN
- K41 pad 5: /TengN_sw -> /TengN_IN
- K42 pad 5: /TengN_sw -> /TengN_IN
- K43 pad 8: /Vsense -> /V_daq+
- K44 pad 8: /Vsense -> /V_daq+
- K45 pad 8: /Vsense -> /V_daq+
- K46 pad 5: /TengN_sw -> /TengN_IN
- K47 pad 5: /TengN_sw -> /TengN_IN
- K48 pad 5: /TengN_sw -> /TengN_IN
- K5 pad 8: /Vsense -> /V_daq+
- K6 pad 5: /TengN_sw -> /TengN_IN
- K7 pad 5: /TengN_sw -> /TengN_IN
- K8 pad 5: /TengN_sw -> /TengN_IN
- K9 pad 5: /TengN_sw -> /TengN_IN
Routing:
- net /Vsense: track 823.7 -> 0.00 mm, vias 1 -> 0
- net /V_daq+: track 30.6 -> 827.7 mm
- net /TengN_sw: track 790.6 -> 0.00 mm, vias 2 -> 0
- net /TengN_IN: track 59.8 -> 773.0 mm, vias 0 -> 2
- net -VCC: track 178.7 -> 0.00 mm, vias 4 -> 0
- net /Dout1: track 135.2 -> 0.00 mm, vias 2 -> 0
- net /Dout2: track 87.5 -> 0.00 mm
- net VCC: track 304.5 -> 227.2 mm, vias 4 -> 2
- net GND: track 769.3 -> 701.4 mm, vias 20 -> 15
- net /V_daq-: track 33.7 -> 0.00 mm
- net /Current_Sense2_IN: track 27.7 -> 0.00 mm
- net /Current_Sense2_OUT: track 26.2 -> 0.00 mm
- net /Current_Sense1_IN: track 24.2 -> 0.00 mm
- net /VNeg: track 18.1 -> 0.00 mm
- net Net-(J4-Pin_1): track 0.00 -> 9.00 mm
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- removed copper zone on B.Cu, net GND
Other:
- board text removed: "-VCC"
- board text removed: "Current Sensor"
- board text removed: "Dout1"
- board text removed: "Dout2"
- board text removed: "GND Current Sensor"
- board text removed: "No Current Sense"
- board text removed: "TIA"
