File: TENG_Loads_PCB/load_automatisation.kicad_sch (KiCad schematic)
At the start: 16 parts, among them J1 1923937, J13 1757242, J2 1757242, J4 PowerIn, U1 AMS1117-5.0

Commit message: Update footprints
Update component footprints, and advancing in the design.
Parts:
- removed C20, C3, C5: 100nF, Capacitor_SMD:C_0805_2012Metric, symbol Device:C
Connections:
- net Din0: now also J1.2; no longer J1.8
- net Din1: now also J1.3; no longer J1.7
- net Din2: now also J1.4; no longer J1.6
- net Din4: now also J1.6; no longer J1.4
- net Din5: now also J1.7; no longer J1.3
- net GND: now also J1.1, J2.2; no longer J1.9, J2.1
- net TengN_IN: now also J1.9; no longer J1.2
- net V_daq+: now also J1.8; no longer J1.1
- net Vin: now also J4.2 (Pin_2); no longer J4.1 (Pin_1)
- new net: J2.1, J4.1 (Pin_1)
Other:
- moved on the sheet: J1, J13, J2, J4, TENG_Connector1, TENG_Connector2
